Commit message: Update description and bringup generated files to be also applicable to mobile robots. Update generated documenation in README files. Add templates for simulation and moveit setup.

File: templates/robot_description/robot_macro.ros2_control.xacro (robot description, xacro)
@@ -15,4 +15,5 @@
           <plugin>mock_components/GenericSystem</plugin>
           <param name="mock_sensor_commands">${mock_sensor_commands}</param>
+          <param name="calculate_dynamics">true</param>
         </xacro:if>
         <xacro:if value="${sim_gazebo_classic}">
@@ -34,6 +35,10 @@
           <param name="initial_value">0.0</param>
         </state_interface>
-        <state_interface name="velocity"/>
-        <state_interface name="acceleration"/>
+        <state_interface name="velocity">
+          <param name="initial_value">0.0</param>
+        </state_interface>
+        <state_interface name="acceleration">
+          <param name="initial_value">0.0</param>
+        </state_interface>
       </joint>
       <joint name="${prefix}joint2">
@@ -45,6 +50,10 @@
           <param name="initial_value">0.0</param>
         </state_interface>
-        <state_interface name="velocity"/>
-        <state_interface name="acceleration"/>
+        <state_interface name="velocity">
+          <param name="initial_value">0.0</param>
+        </state_interface>
+        <state_interface name="acceleration">
+          <param name="initial_value">0.0</param>
+        </state_interface>
       </joint>
       <joint name="${prefix}joint3">
@@ -56,6 +65,10 @@
           <param name="initial_value">0.0</param>
         </state_interface>
-        <state_interface name="velocity"/>
-        <state_interface name="acceleration"/>
+        <state_interface name="velocity">
+          <param name="initial_value">0.0</param>
+        </state_interface>
+        <state_interface name="acceleration">
+          <param name="initial_value">0.0</param>
+        </state_interface>
       </joint>
       <joint name="${prefix}joint4">
@@ -67,6 +80,10 @@
           <param name="initial_value">0.0</param>
         </state_interface>
-        <state_interface name="velocity"/>
-        <state_interface name="acceleration"/>
+        <state_interface name="velocity">
+          <param name="initial_value">0.0</param>
+        </state_interface>
+        <state_interface name="acceleration">
+          <param name="initial_value">0.0</param>
+        </state_interface>
       </joint>
       <joint name="${prefix}joint5">
@@ -78,6 +95,10 @@
           <param name="initial_value">0.0</param>
         </state_interface>
-        <state_interface name="velocity"/>
-        <state_interface name="acceleration"/>
+        <state_interface name="velocity">
+          <param name="initial_value">0.0</param>
+        </state_interface>
+        <state_interface name="acceleration">
+          <param name="initial_value">0.0</param>
+        </state_interface>
       </joint>
       <joint name="${prefix}joint6">
@@ -89,14 +110,30 @@
           <param name="initial_value">0.0</param>
         </state_interface>
-        <state_interface name="velocity"/>
-        <state_interface name="acceleration"/>
+        <state_interface name="velocity">
+          <param name="initial_value">0.0</param>
+        </state_interface>
+        <state_interface name="acceleration">
+          <param name="initial_value">0.0</param>
+        </state_interface>
       </joint>
       <sensor name="tcp_fts_sensor">            <!-- Remove/change sensors as needed -->
-        <state_interface name="fx"/>
-        <state_interface name="fy"/>
-        <state_interface name="fz"/>
-        <state_interface name="tx"/>
-        <state_interface name="ty"/>
-        <state_interface name="tz"/>
+        <state_interface name="fx">
+          <param name="initial_value">0.0</param>
+        </state_interface>
+        <state_interface name="fy">
+          <param name="initial_value">0.0</param>
+        </state_interface>
+        <state_interface name="fz">
+          <param name="initial_value">0.0</param>
+        </state_interface>
+        <state_interface name="tx">
+          <param name="initial_value">0.0</param>
+        </state_interface>
+        <state_interface name="ty">
+          <param name="initial_value">0.0</param>
+        </state_interface>
+        <state_interface name="tz">
+          <param name="initial_value">0.0</param>
+        </state_interface>
         <param name="frame_id">tool0</param>    <!-- Change sensors as needed -->
         <param name="min_fx">-100</param>

File: templates/robot_description/robot_macro.xacro (robot description, xacro)
@@ -3,4 +3,6 @@
   <xacro:include filename="$(find $PKG_NAME$)/urdf/common/inertials.xacro" />
   <xacro:include filename="$(find $PKG_NAME$)/urdf/common/materials.xacro" />
+  <!-- ATTTTTTEEEEENNNNNNNTTTTTIIIIIIOOOOOOONNNNNN -->
+  <!-- If you are dealing with a mobile robot, remove fixing it t the world!! -->
   <xacro:macro name="$ROBOT_NAME$" params="prefix parent *origin">
     <!-- LINKS -->
@@ -14,5 +16,5 @@
         <geometry>
           <cylinder length="0.3" radius="0.3" />
-<!--           <mesh filename="package://$PKG_NAME$/meshes/$ROBOT_NAME$/visual/base_link.dae" /> -->
+<!--           <mesh filename="file://$(find $PKG_NAME$)/meshes/$ROBOT_NAME$/visual/base_link.dae" /> -->
         </geometry>
         <material name="black"/>
@@ -22,5 +24,5 @@
         <geometry>
           <cylinder length="0.3" radius="0.3" />
-<!--           <mesh filename="package://$PKG_NAME$/meshes/$ROBOT_NAME$/collision/base_link.stl" /> -->
+<!--           <mesh filename="file://$(find $PKG_NAME$)/meshes/$ROBOT_NAME$/collision/base_link.stl" /> -->
         </geometry>
       </collision>
@@ -35,5 +37,5 @@
         <geometry>
           <cylinder length="0.3" radius="0.15" />
-<!--           <mesh filename="package://$PKG_NAME$/meshes/$ROBOT_NAME$/visual/link1.dae" /> -->
+<!--           <mesh filename="file://$(find $PKG_NAME$)/meshes/$ROBOT_NAME$/visual/link1.dae" /> -->
         </geometry>
         <material name="blue"/>
@@ -43,5 +45,5 @@
         <geometry>
           <cylinder length="0.3" radius="0.15" />
-<!--           <mesh filename="package://$PKG_NAME$/meshes/$ROBOT_NAME$/collision/link1.stl" /> -->
+<!--           <mesh filename="file://$(find $PKG_NAME$)/meshes/$ROBOT_NAME$/collision/link1.stl" /> -->
         </geometry>
         <material name="green"/>
@@ -57,5 +59,5 @@
         <geometry>
           <cylinder length="0.8" radius="0.15" />
-<!--           <mesh filename="package://$PKG_NAME$/meshes/$ROBOT_NAME$/visual/link2.dae" /> -->
+<!--           <mesh filename="file://$(find $PKG_NAME$)/meshes/$ROBOT_NAME$/visual/link2.dae" /> -->
         </geometry>
         <material name="grey"/>
@@ -65,5 +67,5 @@
         <geometry>
           <cylinder length="0.8" radius="0.15" />
-<!--           <mesh filename="package://$PKG_NAME$/meshes/$ROBOT_NAME$/collision/link2.stl"  /> -->
+<!--           <mesh filename="file://$(find $PKG_NAME$)/meshes/$ROBOT_NAME$/collision/link2.stl"  /> -->
         </geometry>
       </collision>
@@ -78,5 +80,5 @@
         <geometry>
           <cylinder length="0.5" radius="0.10" />
-<!--           <mesh filename="package://$PKG_NAME$/meshes/$ROBOT_NAME$/visual/link3.dae" /> -->
+<!--           <mesh filename="file://$(find $PKG_NAME$)/meshes/$ROBOT_NAME$/visual/link3.dae" /> -->
         </geometry>
         <material name="orange"/>
@@ -86,5 +88,5 @@
         <geometry>
           <cylinder length="0.5" radius="0.10" />
-<!--           <mesh filename="package://$PKG_NAME$/meshes/$ROBOT_NAME$/collision/link3.stl"  /> -->
+<!--           <mesh filename="file://$(find $PKG_NAME$)/meshes/$ROBOT_NAME$/collision/link3.stl"  /> -->
         </geometry>
       </collision>
@@ -99,5 +101,5 @@
         <geometry>
           <cylinder length="0.1" radius="0.2" />
-<!--           <mesh filename="package://$PKG_NAME$/meshes/$ROBOT_NAME$/visual/link4.dae" /> -->
+<!--           <mesh filename="file://$(find $PKG_NAME$)/meshes/$ROBOT_NAME$/visual/link4.dae" /> -->
         </geometry>
         <material name="brown"/>
@@ -107,5 +109,5 @@
         <geometry>
           <cylinder length="0.1" radius="0.2" />
-<!--           <mesh filename="package://$PKG_NAME$/meshes/$ROBOT_NAME$/collision/link4.stl"  /> -->
+<!--           <mesh filename="file://$(find $PKG_NAME$)/meshes/$ROBOT_NAME$/collision/link4.stl"  /> -->
         </geometry>
       </collision>
@@ -120,5 +122,5 @@
         <geometry>
           <cylinder length="0.2" radius="0.1" />
-<!--           <mesh filename="package://$PKG_NAME$/meshes/$ROBOT_NAME$/visual/link5.dae" /> -->
+<!--           <mesh filename="file://$(find $PKG_NAME$)/meshes/$ROBOT_NAME$/visual/link5.dae" /> -->
         </geometry>
         <material name="red"/>
@@ -128,5 +130,5 @@
         <geometry>
           <cylinder length="0.2" radius="0.1" />
-<!--           <mesh filename="package://$PKG_NAME$/meshes/$ROBOT_NAME$/collision/link5.stl" /> -->
+<!--           <mesh filename="file://$(find $PKG_NAME$)/meshes/$ROBOT_NAME$/collision/link5.stl" /> -->
         </geometry>
       </collision>
@@ -141,5 +143,5 @@
         <geometry>
           <cylinder length="0.05" radius="0.1" />
-<!--           <mesh filename="package://$PKG_NAME$/meshes/$ROBOT_NAME$/visual/link6.dae" /> -->
+<!--           <mesh filename="file://$(find $PKG_NAME$)/meshes/$ROBOT_NAME$/visual/link6.dae" /> -->
         </geometry>
         <material name="white"/>
@@ -149,5 +151,5 @@
         <geometry>
           <cylinder length="0.05" radius="0.1" />
-<!--           <mesh filename="package://$PKG_NAME$/meshes/$ROBOT_NAME$/collision/link6.stl" /> -->
+<!--           <mesh filename="file://$(find $PKG_NAME$)/meshes/$ROBOT_NAME$/collision/link6.stl" /> -->
         </geometry>
       </collision>
